File: FPGA_decoup_capacitors.kicad_sch (KiCad schematic)
At the start: 32 parts

Commit message: Added footprints to symbols
Some nice light work
Parts:
- C20, C21, C22, C23, C24, C25, C26, C27, C28, C29, C30, C31, C32, C33, C34, C35, C36, C37, C38, C39, C40, C41, C42, C43, C44, C45, C46, C47, C48, C49, C50, C51: footprint (none) -> Capacitor_SMD:C_1206_3216Metric
Changed lines of the file:
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@@
       (effects (font (size 1.27 1.27)) (justify left))
     )
-    (property "Footprint" "" (at 82.2452 93.98 0)
+    (property "Footprint" "Capacitor_SMD:C_1206_3216Metric" (at 82.2452 93.98 0)
       (effects (font (size 1.27 1.27)) hide)
     )
@@
       (effects (font (size 1.27 1.27)) (justify left))
     )
-    (property "Footprint" "" (at 92.4052 93.98 0)
+    (property "Footprint" "Capacitor_SMD:C_1206_3216Metric" (at 92.4052 93.98 0)
       (effects (font (size 1.27 1.27)) hide)
     )
@@
       (effects (font (size 1.27 1.27)) (justify left))
     )
-    (property "Footprint" "" (at 105.1052 93.98 0)
+    (property "Footprint" "Capacitor_SMD:C_1206_3216Metric" (at 105.1052 93.98 0)
       (effects (font (size 1.27 1.27)) hide)
     )
@@
       (effects (font (size 1.27 1.27)) (justify left))
     )
-    (property "Footprint" "" (at 110.1852 116.84 0)
+    (property "Footprint" "Capacitor_SMD:C_1206_3216Metric" (at 110.1852 116.84 0)
       (effects (font (size 1.27 1.27)) hide)
     )
@@
       (effects (font (size 1.27 1.27)) (justify left))
     )
-    (property "Footprint" "" (at 79.7052 116.84 0)
+    (property "Footprint" "Capacitor_SMD:C_1206_3216Metric" (at 79.7052 116.84 0)
       (effects (font (size 1.27 1.27)) hide)
     )
@@
       (effects (font (size 1.27 1.27)) (justify left))
     )
-    (property "Footprint" "" (at 94.9452 48.26 0)
+    (property "Footprint" "Capacitor_SMD:C_1206_3216Metric" (at 94.9452 48.26 0)
       (effects (font (size 1.27 1.27)) hide)
     )
@@
       (effects (font (size 1.27 1.27)) (justify left))
     )
-    (property "Footprint" "" (at 88.5952 48.26 0)
+    (property "Footprint" "Capacitor_SMD:C_1206_3216Metric" (at 88.5952 48.26 0)
       (effects (font (size 1.27 1.27)) hide)
     )
@@
       (effects (font (size 1.27 1.27)) (justify left))
     )
-    (property "Footprint" "" (at 122.8852 116.84 0)
+    (property "Footprint" "Capacitor_SMD:C_1206_3216Metric" (at 122.8852 116.84 0)
       (effects (font (size 1.27 1.27)) hide)
     )
@@
       (effects (font (size 1.27 1.27)) (justify left))
     )
-    (property "Footprint" "" (at 144.4752 48.26 0)
+    (property "Footprint" "Capacitor_SMD:C_1206_3216Metric" (at 144.4752 48.26 0)
       (effects (font (size 1.27 1.27)) hide)
     )
@@
       (effects (font (size 1.27 1.27)) (justify left))
     )
-    (property "Footprint" "" (at 150.8252 48.26 0)
+    (property "Footprint" "Capacitor_SMD:C_1206_3216Metric" (at 150.8252 48.26 0)
       (effects (font (size 1.27 1.27)) hide)
     )
@@
       (effects (font (size 1.27 1.27)) (justify left))
     )
-    (property "Footprint" "" (at 80.9752 71.12 0)
+    (property "Footprint" "Capacitor_SMD:C_1206_3216Metric" (at 80.9752 71.12 0)
       (effects (font (size 1.27 1.27)) hide)
     )
@@
       (effects (font (size 1.27 1.27)) (justify left))
     )
-    (property "Footprint" "" (at 64.4652 71.12 0)
+    (property "Footprint" "Capacitor_SMD:C_1206_3216Metric" (at 64.4652 71.12 0)
       (effects (font (size 1.27 1.27)) hide)
     )
@@
       (effects (font (size 1.27 1.27)) (justify left))
     )
-    (property "Footprint" "" (at 64.4652 93.98 0)
+    (property "Footprint" "Capacitor_SMD:C_1206_3216Metric" (at 64.4652 93.98 0)
       (effects (font (size 1.27 1.27)) hide)
     )
@@
       (effects (font (size 1.27 1.27)) (justify left))
     )
-    (property "Footprint" "" (at 75.8952 48.26 0)
+    (property "Footprint" "Capacitor_SMD:C_1206_3216Metric" (at 75.8952 48.26 0)
       (effects (font (size 1.27 1.27)) hide)
     )
@@
       (effects (font (size 1.27 1.27)) (justify left))
     )
-    (property "Footprint" "" (at 107.6452 48.26 0)
+    (property "Footprint" "Capacitor_SMD:C_1206_3216Metric" (at 107.6452 48.26 0)
       (effects (font (size 1.27 1.27)) hide)
     )
@@
       (effects (font (size 1.27 1.27)) (justify left))
     )
-    (property "Footprint" "" (at 98.7552 93.98 0)
+    (property "Footprint" "Capacitor_SMD:C_1206_3216Metric" (at 98.7552 93.98 0)
       (effects (font (size 1.27 1.27)) hide)
     )
@@
       (effects (font (size 1.27 1.27)) (justify left))
     )
-    (property "Footprint" "" (at 64.4652 48.26 0)
+    (property "Footprint" "Capacitor_SMD:C_1206_3216Metric" (at 64.4652 48.26 0)
       (effects (font (size 1.27 1.27)) hide)
     )
@@
       (effects (font (size 1.27 1.27)) (justify left))
     )
-    (property "Footprint" "" (at 119.0752 48.26 0)
+    (property "Footprint" "Capacitor_SMD:C_1206_3216Metric" (at 119.0752 48.26 0)
       (effects (font (size 1.27 1.27)) hide)
     )
@@
       (effects (font (size 1.27 1.27)) (justify left))
     )
-    (property "Footprint" "" (at 131.7752 48.26 0)
+    (property "Footprint" "Capacitor_SMD:C_1206_3216Metric" (at 131.7752 48.26 0)
       (effects (font (size 1.27 1.27)) hide)
     )
@@
       (effects (font (size 1.27 1.27)) (justify left))
     )
-    (property "Footprint" "" (at 129.2352 116.84 0)
+    (property "Footprint" "Capacitor_SMD:C_1206_3216Metric" (at 129.2352 116.84 0)
       (effects (font (size 1.27 1.27)) hide)
     )
@@
       (effects (font (size 1.27 1.27)) (justify left))
     )
-    (property "Footprint" "" (at 75.8952 93.98 0)
+    (property "Footprint" "Capacitor_SMD:C_1206_3216Metric" (at 75.8952 93.98 0)
       (effects (font (size 1.27 1.27)) hide)
     )
@@
       (effects (font (size 1.27 1.27)) (justify left))
     )
-    (property "Footprint" "" (at 125.4252 48.26 0)
+    (property "Footprint" "Capacitor_SMD:C_1206_3216Metric" (at 125.4252 48.26 0)
       (effects (font (size 1.27 1.27)) hide)
     )
@@
       (effects (font (size 1.27 1.27)) (justify left))
     )
-    (property "Footprint" "" (at 157.1752 48.26 0)
+    (property "Footprint" "Capacitor_SMD:C_1206_3216Metric" (at 157.1752 48.26 0)
       (effects (font (size 1.27 1.27)) hide)
     )
@@
       (effects (font (size 1.27 1.27)) (justify left))
     )
-    (property "Footprint" "" (at 93.6752 116.84 0)
+    (property "Footprint" "Capacitor_SMD:C_1206_3216Metric" (at 93.6752 116.84 0)
       (effects (font (size 1.27 1.27)) hide)
     )
@@
       (effects (font (size 1.27 1.27)) (justify left))
     )
-    (property "Footprint" "" (at 116.5352 116.84 0)
+    (property "Footprint" "Capacitor_SMD:C_1206_3216Metric" (at 116.5352 116.84 0)
       (effects (font (size 1.27 1.27)) hide)
     )
@@
       (effects (font (size 1.27 1.27)) (justify left))
     )
-    (property "Footprint" "" (at 138.1252 48.26 0)
+    (property "Footprint" "Capacitor_SMD:C_1206_3216Metric" (at 138.1252 48.26 0)
       (effects (font (size 1.27 1.27)) hide)
     )
@@
       (effects (font (size 1.27 1.27)) (justify left))
     )
-    (property "Footprint" "" (at 163.5252 48.26 0)
+    (property "Footprint" "Capacitor_SMD:C_1206_3216Metric" (at 163.5252 48.26 0)
       (effects (font (size 1.27 1.27)) hide)
     )
@@
       (effects (font (size 1.27 1.27)) (justify left))
     )
-    (property "Footprint" "" (at 64.4652 116.84 0)
+    (property "Footprint" "Capacitor_SMD:C_1206_3216Metric" (at 64.4652 116.84 0)
       (effects (font (size 1.27 1.27)) hide)
     )
@@
       (effects (font (size 1.27 1.27)) (justify left))
     )
-    (property "Footprint" "" (at 101.2952 48.26 0)
+    (property "Footprint" "Capacitor_SMD:C_1206_3216Metric" (at 101.2952 48.26 0)
       (effects (font (size 1.27 1.27)) hide)
     )
@@
       (effects (font (size 1.27 1.27)) (justify left))
     )
-    (property "Footprint" "" (at 100.0252 116.84 0)
+    (property "Footprint" "Capacitor_SMD:C_1206_3216Metric" (at 100.0252 116.84 0)
       (effects (font (size 1.27 1.27)) hide)
     )
@@
       (effects (font (size 1.27 1.27)) (justify left))
     )
-    (property "Footprint" "" (at 82.2452 48.26 0)
+    (property "Footprint" "Capacitor_SMD:C_1206_3216Metric" (at 82.2452 48.26 0)
       (effects (font (size 1.27 1.27)) hide)
     )
@@
       (effects (font (size 1.27 1.27)) (justify left))
     )
-    (property "Footprint" "" (at 74.6252 71.12 0)
-      (effects (font (size 1.27 1.27)) hide)
-    )
+    (property "Footprint" "Capacitor_SMD:C_1206_3216Metric" (at 74.6252 71.12 0)
+      (effects (font (size 1.27 1.27)) hide)
+    )

Commit message: Changed Reistor and Capacitor size fomr 1206 to 0805
Parts:
- C20, C21, C22, C23, C24, C25, C26, C27, C28, C29, C30, C31, C32, C33, C34, C35, C36, C37, C38, C39, C40, C41, C42, C43, C44, C45, C46, C47, C48, C49, C50, C51: footprint Capacitor_SMD:C_1206_3216Metric -> Capacitor_SMD:C_0805_2012Metric
Changed lines of the file:
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@@
       (effects (font (size 1.27 1.27)) (justify left))
     )
-    (property "Footprint" "Capacitor_SMD:C_1206_3216Metric" (at 82.2452 93.98 0)
+    (property "Footprint" "Capacitor_SMD:C_0805_2012Metric" (at 82.2452 93.98 0)
       (effects (font (size 1.27 1.27)) hide)
     )
@@
       (effects (font (size 1.27 1.27)) (justify left))
     )
-    (property "Footprint" "Capacitor_SMD:C_1206_3216Metric" (at 92.4052 93.98 0)
+    (property "Footprint" "Capacitor_SMD:C_0805_2012Metric" (at 92.4052 93.98 0)
       (effects (font (size 1.27 1.27)) hide)
     )
@@
       (effects (font (size 1.27 1.27)) (justify left))
     )
-    (property "Footprint" "Capacitor_SMD:C_1206_3216Metric" (at 105.1052 93.98 0)
+    (property "Footprint" "Capacitor_SMD:C_0805_2012Metric" (at 105.1052 93.98 0)
       (effects (font (size 1.27 1.27)) hide)
     )
@@
       (effects (font (size 1.27 1.27)) (justify left))
     )
-    (property "Footprint" "Capacitor_SMD:C_1206_3216Metric" (at 110.1852 116.84 0)
+    (property "Footprint" "Capacitor_SMD:C_0805_2012Metric" (at 110.1852 116.84 0)
       (effects (font (size 1.27 1.27)) hide)
     )
@@
       (effects (font (size 1.27 1.27)) (justify left))
     )
-    (property "Footprint" "Capacitor_SMD:C_1206_3216Metric" (at 79.7052 116.84 0)
+    (property "Footprint" "Capacitor_SMD:C_0805_2012Metric" (at 79.7052 116.84 0)
       (effects (font (size 1.27 1.27)) hide)
     )
@@
       (effects (font (size 1.27 1.27)) (justify left))
     )
-    (property "Footprint" "Capacitor_SMD:C_1206_3216Metric" (at 94.9452 48.26 0)
+    (property "Footprint" "Capacitor_SMD:C_0805_2012Metric" (at 94.9452 48.26 0)
       (effects (font (size 1.27 1.27)) hide)
     )
@@
       (effects (font (size 1.27 1.27)) (justify left))
     )
-    (property "Footprint" "Capacitor_SMD:C_1206_3216Metric" (at 88.5952 48.26 0)
+    (property "Footprint" "Capacitor_SMD:C_0805_2012Metric" (at 88.5952 48.26 0)
       (effects (font (size 1.27 1.27)) hide)
     )
@@
       (effects (font (size 1.27 1.27)) (justify left))
     )
-    (property "Footprint" "Capacitor_SMD:C_1206_3216Metric" (at 122.8852 116.84 0)
+    (property "Footprint" "Capacitor_SMD:C_0805_2012Metric" (at 122.8852 116.84 0)
       (effects (font (size 1.27 1.27)) hide)
     )
@@
       (effects (font (size 1.27 1.27)) (justify left))
     )
-    (property "Footprint" "Capacitor_SMD:C_1206_3216Metric" (at 144.4752 48.26 0)
+    (property "Footprint" "Capacitor_SMD:C_0805_2012Metric" (at 144.4752 48.26 0)
       (effects (font (size 1.27 1.27)) hide)
     )
@@
       (effects (font (size 1.27 1.27)) (justify left))
     )
-    (property "Footprint" "Capacitor_SMD:C_1206_3216Metric" (at 150.8252 48.26 0)
+    (property "Footprint" "Capacitor_SMD:C_0805_2012Metric" (at 150.8252 48.26 0)
       (effects (font (size 1.27 1.27)) hide)
     )
@@
       (effects (font (size 1.27 1.27)) (justify left))
     )
-    (property "Footprint" "Capacitor_SMD:C_1206_3216Metric" (at 80.9752 71.12 0)
+    (property "Footprint" "Capacitor_SMD:C_0805_2012Metric" (at 80.9752 71.12 0)
       (effects (font (size 1.27 1.27)) hide)
     )
@@
       (effects (font (size 1.27 1.27)) (justify left))
     )
-    (property "Footprint" "Capacitor_SMD:C_1206_3216Metric" (at 64.4652 71.12 0)
+    (property "Footprint" "Capacitor_SMD:C_0805_2012Metric" (at 64.4652 71.12 0)
       (effects (font (size 1.27 1.27)) hide)
     )
@@
       (effects (font (size 1.27 1.27)) (justify left))
     )
-    (property "Footprint" "Capacitor_SMD:C_1206_3216Metric" (at 64.4652 93.98 0)
+    (property "Footprint" "Capacitor_SMD:C_0805_2012Metric" (at 64.4652 93.98 0)
       (effects (font (size 1.27 1.27)) hide)
     )
@@
       (effects (font (size 1.27 1.27)) (justify left))
     )
-    (property "Footprint" "Capacitor_SMD:C_1206_3216Metric" (at 75.8952 48.26 0)
+    (property "Footprint" "Capacitor_SMD:C_0805_2012Metric" (at 75.8952 48.26 0)
       (effects (font (size 1.27 1.27)) hide)
     )
@@
       (effects (font (size 1.27 1.27)) (justify left))
     )
-    (property "Footprint" "Capacitor_SMD:C_1206_3216Metric" (at 107.6452 48.26 0)
+    (property "Footprint" "Capacitor_SMD:C_0805_2012Metric" (at 107.6452 48.26 0)
       (effects (font (size 1.27 1.27)) hide)
     )
@@
       (effects (font (size 1.27 1.27)) (justify left))
     )
-    (property "Footprint" "Capacitor_SMD:C_1206_3216Metric" (at 98.7552 93.98 0)
+    (property "Footprint" "Capacitor_SMD:C_0805_2012Metric" (at 98.7552 93.98 0)
       (effects (font (size 1.27 1.27)) hide)
     )
@@
       (effects (font (size 1.27 1.27)) (justify left))
     )
-    (property "Footprint" "Capacitor_SMD:C_1206_3216Metric" (at 64.4652 48.26 0)
+    (property "Footprint" "Capacitor_SMD:C_0805_2012Metric" (at 64.4652 48.26 0)
       (effects (font (size 1.27 1.27)) hide)
     )
@@
       (effects (font (size 1.27 1.27)) (justify left))
     )
-    (property "Footprint" "Capacitor_SMD:C_1206_3216Metric" (at 119.0752 48.26 0)
+    (property "Footprint" "Capacitor_SMD:C_0805_2012Metric" (at 119.0752 48.26 0)
       (effects (font (size 1.27 1.27)) hide)
     )
@@
       (effects (font (size 1.27 1.27)) (justify left))
     )
-    (property "Footprint" "Capacitor_SMD:C_1206_3216Metric" (at 131.7752 48.26 0)
+    (property "Footprint" "Capacitor_SMD:C_0805_2012Metric" (at 131.7752 48.26 0)
       (effects (font (size 1.27 1.27)) hide)
     )
@@
       (effects (font (size 1.27 1.27)) (justify left))
     )
-    (property "Footprint" "Capacitor_SMD:C_1206_3216Metric" (at 129.2352 116.84 0)
+    (property "Footprint" "Capacitor_SMD:C_0805_2012Metric" (at 129.2352 116.84 0)
       (effects (font (size 1.27 1.27)) hide)
     )
@@
       (effects (font (size 1.27 1.27)) (justify left))
     )
-    (property "Footprint" "Capacitor_SMD:C_1206_3216Metric" (at 75.8952 93.98 0)
+    (property "Footprint" "Capacitor_SMD:C_0805_2012Metric" (at 75.8952 93.98 0)
       (effects (font (size 1.27 1.27)) hide)
     )
@@
       (effects (font (size 1.27 1.27)) (justify left))
     )
-    (property "Footprint" "Capacitor_SMD:C_1206_3216Metric" (at 125.4252 48.26 0)
+    (property "Footprint" "Capacitor_SMD:C_0805_2012Metric" (at 125.4252 48.26 0)
       (effects (font (size 1.27 1.27)) hide)
     )
@@
       (effects (font (size 1.27 1.27)) (justify left))
     )
-    (property "Footprint" "Capacitor_SMD:C_1206_3216Metric" (at 157.1752 48.26 0)
+    (property "Footprint" "Capacitor_SMD:C_0805_2012Metric" (at 157.1752 48.26 0)
       (effects (font (size 1.27 1.27)) hide)
     )
@@
       (effects (font (size 1.27 1.27)) (justify left))
     )
-    (property "Footprint" "Capacitor_SMD:C_1206_3216Metric" (at 93.6752 116.84 0)
+    (property "Footprint" "Capacitor_SMD:C_0805_2012Metric" (at 93.6752 116.84 0)
       (effects (font (size 1.27 1.27)) hide)
     )
@@
       (effects (font (size 1.27 1.27)) (justify left))
     )
-    (property "Footprint" "Capacitor_SMD:C_1206_3216Metric" (at 116.5352 116.84 0)
+    (property "Footprint" "Capacitor_SMD:C_0805_2012Metric" (at 116.5352 116.84 0)
       (effects (font (size 1.27 1.27)) hide)
     )
@@
       (effects (font (size 1.27 1.27)) (justify left))
     )
-    (property "Footprint" "Capacitor_SMD:C_1206_3216Metric" (at 138.1252 48.26 0)
+    (property "Footprint" "Capacitor_SMD:C_0805_2012Metric" (at 138.1252 48.26 0)
       (effects (font (size 1.27 1.27)) hide)
     )
@@
       (effects (font (size 1.27 1.27)) (justify left))
     )
-    (property "Footprint" "Capacitor_SMD:C_1206_3216Metric" (at 163.5252 48.26 0)
+    (property "Footprint" "Capacitor_SMD:C_0805_2012Metric" (at 163.5252 48.26 0)
       (effects (font (size 1.27 1.27)) hide)
     )
@@
       (effects (font (size 1.27 1.27)) (justify left))
     )
-    (property "Footprint" "Capacitor_SMD:C_1206_3216Metric" (at 64.4652 116.84 0)
+    (property "Footprint" "Capacitor_SMD:C_0805_2012Metric" (at 64.4652 116.84 0)
       (effects (font (size 1.27 1.27)) hide)
     )
@@
       (effects (font (size 1.27 1.27)) (justify left))
     )
-    (property "Footprint" "Capacitor_SMD:C_1206_3216Metric" (at 101.2952 48.26 0)
+    (property "Footprint" "Capacitor_SMD:C_0805_2012Metric" (at 101.2952 48.26 0)
       (effects (font (size 1.27 1.27)) hide)
     )
@@
       (effects (font (size 1.27 1.27)) (justify left))
     )
-    (property "Footprint" "Capacitor_SMD:C_1206_3216Metric" (at 100.0252 116.84 0)
+    (property "Footprint" "Capacitor_SMD:C_0805_2012Metric" (at 100.0252 116.84 0)
       (effects (font (size 1.27 1.27)) hide)
     )
@@
       (effects (font (size 1.27 1.27)) (justify left))
     )
-    (property "Footprint" "Capacitor_SMD:C_1206_3216Metric" (at 82.2452 48.26 0)
+    (property "Footprint" "Capacitor_SMD:C_0805_2012Metric" (at 82.2452 48.26 0)
       (effects (font (size 1.27 1.27)) hide)
     )
@@
       (effects (font (size 1.27 1.27)) (justify left))
     )
-    (property "Footprint" "Capacitor_SMD:C_1206_3216Metric" (at 74.6252 71.12 0)
-      (effects (font (size 1.27 1.27)) hide)
-    )
+    (property "Footprint" "Capacitor_SMD:C_0805_2012Metric" (at 74.6252 71.12 0)
+      (effects (font (size 1.27 1.27)) hide)
+    )
