File: FPGA_decoup_capacitors.kicad_sch (KiCad schematic)
At the start: 32 parts

Commit message: Resized Capacitors
Parts:
- C20: footprint Capacitor_SMD:C_0805_2012Metric -> T520V337M2R5ATE025:CAPMP7.6X4.3_1.9N_KEM
- C27, C28, C29, C30, C31, C32, C33, C34, C36, C37, C41, C42, C43, C48, C49, C50, C51: footprint Capacitor_SMD:C_0805_2012Metric -> Capacitor_SMD:C_0603_1608Metric
Changed lines of the file:
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@@
       (effects (font (size 1.27 1.27)) (justify left))
     )
-    (property "Footprint" "Capacitor_SMD:C_0805_2012Metric" (at 92.4052 93.98 0)
+    (property "Footprint" "Capacitor_SMD:C_0603_1608Metric" (at 92.4052 93.98 0)
       (effects (font (size 1.27 1.27)) hide)
     )
@@
       (effects (font (size 1.27 1.27)) (justify left))
     )
-    (property "Footprint" "Capacitor_SMD:C_0805_2012Metric" (at 105.1052 93.98 0)
+    (property "Footprint" "Capacitor_SMD:C_0603_1608Metric" (at 105.1052 93.98 0)
       (effects (font (size 1.27 1.27)) hide)
     )
@@
       (effects (font (size 1.27 1.27)) (justify left))
     )
-    (property "Footprint" "Capacitor_SMD:C_0805_2012Metric" (at 110.1852 116.84 0)
+    (property "Footprint" "Capacitor_SMD:C_0603_1608Metric" (at 110.1852 116.84 0)
       (effects (font (size 1.27 1.27)) hide)
     )
@@
       (effects (font (size 1.27 1.27)) (justify left))
     )
-    (property "Footprint" "Capacitor_SMD:C_0805_2012Metric" (at 122.8852 116.84 0)
+    (property "Footprint" "Capacitor_SMD:C_0603_1608Metric" (at 122.8852 116.84 0)
       (effects (font (size 1.27 1.27)) hide)
     )
@@
       (effects (font (size 1.27 1.27)) (justify left))
     )
-    (property "Footprint" "Capacitor_SMD:C_0805_2012Metric" (at 144.4752 48.26 0)
+    (property "Footprint" "Capacitor_SMD:C_0603_1608Metric" (at 144.4752 48.26 0)
       (effects (font (size 1.27 1.27)) hide)
     )
@@
       (effects (font (size 1.27 1.27)) (justify left))
     )
-    (property "Footprint" "Capacitor_SMD:C_0805_2012Metric" (at 150.8252 48.26 0)
+    (property "Footprint" "Capacitor_SMD:C_0603_1608Metric" (at 150.8252 48.26 0)
       (effects (font (size 1.27 1.27)) hide)
     )
@@
       (effects (font (size 1.27 1.27)) (justify left))
     )
-    (property "Footprint" "Capacitor_SMD:C_0805_2012Metric" (at 80.9752 71.12 0)
+    (property "Footprint" "Capacitor_SMD:C_0603_1608Metric" (at 80.9752 71.12 0)
       (effects (font (size 1.27 1.27)) hide)
     )
@@
       (effects (font (size 1.27 1.27)) (justify left))
     )
-    (property "Footprint" "Capacitor_SMD:C_0805_2012Metric" (at 98.7552 93.98 0)
+    (property "Footprint" "Capacitor_SMD:C_0603_1608Metric" (at 98.7552 93.98 0)
       (effects (font (size 1.27 1.27)) hide)
     )
@@
       (effects (font (size 1.27 1.27)) (justify left))
     )
-    (property "Footprint" "Capacitor_SMD:C_0805_2012Metric" (at 64.4652 48.26 0)
+    (property "Footprint" "T520V337M2R5ATE025:CAPMP7.6X4.3_1.9N_KEM" (at 64.4652 48.26 0)
       (effects (font (size 1.27 1.27)) hide)
     )
@@
       (effects (font (size 1.27 1.27)) (justify left))
     )
-    (property "Footprint" "Capacitor_SMD:C_0805_2012Metric" (at 119.0752 48.26 0)
+    (property "Footprint" "Capacitor_SMD:C_0603_1608Metric" (at 119.0752 48.26 0)
       (effects (font (size 1.27 1.27)) hide)
     )
@@
       (effects (font (size 1.27 1.27)) (justify left))
     )
-    (property "Footprint" "Capacitor_SMD:C_0805_2012Metric" (at 131.7752 48.26 0)
+    (property "Footprint" "Capacitor_SMD:C_0603_1608Metric" (at 131.7752 48.26 0)
       (effects (font (size 1.27 1.27)) hide)
     )
@@
       (effects (font (size 1.27 1.27)) (justify left))
     )
-    (property "Footprint" "Capacitor_SMD:C_0805_2012Metric" (at 129.2352 116.84 0)
+    (property "Footprint" "Capacitor_SMD:C_0603_1608Metric" (at 129.2352 116.84 0)
       (effects (font (size 1.27 1.27)) hide)
     )
@@
       (effects (font (size 1.27 1.27)) (justify left))
     )
-    (property "Footprint" "Capacitor_SMD:C_0805_2012Metric" (at 125.4252 48.26 0)
+    (property "Footprint" "Capacitor_SMD:C_0603_1608Metric" (at 125.4252 48.26 0)
       (effects (font (size 1.27 1.27)) hide)
     )
@@
       (effects (font (size 1.27 1.27)) (justify left))
     )
-    (property "Footprint" "Capacitor_SMD:C_0805_2012Metric" (at 157.1752 48.26 0)
+    (property "Footprint" "Capacitor_SMD:C_0603_1608Metric" (at 157.1752 48.26 0)
       (effects (font (size 1.27 1.27)) hide)
     )
@@
       (effects (font (size 1.27 1.27)) (justify left))
     )
-    (property "Footprint" "Capacitor_SMD:C_0805_2012Metric" (at 116.5352 116.84 0)
+    (property "Footprint" "Capacitor_SMD:C_0603_1608Metric" (at 116.5352 116.84 0)
       (effects (font (size 1.27 1.27)) hide)
     )
@@
       (effects (font (size 1.27 1.27)) (justify left))
     )
-    (property "Footprint" "Capacitor_SMD:C_0805_2012Metric" (at 138.1252 48.26 0)
+    (property "Footprint" "Capacitor_SMD:C_0603_1608Metric" (at 138.1252 48.26 0)
       (effects (font (size 1.27 1.27)) hide)
     )
@@
       (effects (font (size 1.27 1.27)) (justify left))
     )
-    (property "Footprint" "Capacitor_SMD:C_0805_2012Metric" (at 163.5252 48.26 0)
+    (property "Footprint" "Capacitor_SMD:C_0603_1608Metric" (at 163.5252 48.26 0)
       (effects (font (size 1.27 1.27)) hide)
     )
@@
       (effects (font (size 1.27 1.27)) (justify left))
     )
-    (property "Footprint" "Capacitor_SMD:C_0805_2012Metric" (at 74.6252 71.12 0)
-      (effects (font (size 1.27 1.27)) hide)
-    )
+    (property "Footprint" "Capacitor_SMD:C_0603_1608Metric" (at 74.6252 71.12 0)
+      (effects (font (size 1.27 1.27)) hide)
+    )
