File: _autosave-PSU.kicad_sch (KiCad schematic)
At the start: 34 parts, among them U1 TPS54325, U2 TSP54294

Commit message: Finish Routing of PSU
Connections:
- net at R7.1, R8.2: no longer U2.10 (VFB2)
Changed lines of the file:
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@@
     (stroke (width 0) (type default))
   )
-  (wire (pts (xy 203.2 135.89) (xy 166.37 135.89))
+  (wire (pts (xy 203.2 135.89) (xy 240.03 135.89))
     (stroke (width 0) (type default))
   )
